Commit message: latest using SBL PPO and new negative reward functions

File: src/model/assets/lynx.urdf (robot description, URDF)
Before this commit: robot a4wd1, 6 links, 5 joints
Joints:
- joint joint_fl: limit lower=-1000 upper=1000 effort=10 velocity=50 -> effort=20 velocity=50; type revolute -> continuous
- joint joint_fr: limit lower=-1000 upper=1000 effort=10 velocity=50 -> effort=20 velocity=50; type revolute -> continuous
- joint joint_rl: limit lower=-1000 upper=1000 effort=10 velocity=50 -> effort=20 velocity=50; type revolute -> continuous
- joint joint_rr: limit lower=-1000 upper=1000 effort=10 velocity=50 -> effort=20 velocity=50; type revolute -> continuous
